Commit message: fixed wrong wheel offset from base link origin

File: urdf/volksbot.urdf.xacro (robot description, xacro)
@@ -10,5 +10,5 @@
   <xacro:property name="axis_length" value="0.41" />
   <xacro:property name="wheel_x_offset" value="0.225" />
-  <xacro:property name="wheel_z_offset" value="0.0" />
+  <xacro:property name="wheel_z_offset" value="-0.0275" />
   <xacro:property name="turning_adaptation" value="0.95" />
   <xacro:property name="base_mass" value="10" />
@@ -93,5 +93,6 @@
   </link>
   <joint name="base_footprint_joint" type="fixed">
-    <origin xyz="0 0 ${-wheel_z_offset + wheel_radius}" rpy="0 0 0" />
+    <!-- base link has 5cm clearence from ground and height of 15.5cm -->
+    <origin xyz="0 0 ${0.155/2 + 0.05}" rpy="0 0 0" />
     <parent link="base_footprint"/>
     <child link="base_link" />

Commit message: base link urdf with parameters

File: urdf/volksbot.urdf.xacro (robot description, xacro)
@@ -14,9 +14,12 @@
   <xacro:property name="base_mass" value="10" />
   <xacro:property name="wheel_mass" value="0.25" />
+  <xacro:property name="base_link_length" value="0.55"/>
+  <xacro:property name="base_link_width" value="0.32"/>
+  <xacro:property name="base_link_height" value="0.155"/>
   <link name="base_link">
     <visual>
       <origin xyz="0 0 0" rpy="0 0 0" />
       <geometry>
-        <!--<box size="0.55 0.32 0.155" />-->
+        <!--<box size="${base_link_length} ${base_link_width} ${base_link_height}" />-->
         <mesh filename="package://volksbot_driver/meshes/base.stl"/>
       </geometry>
@@ -28,9 +31,9 @@
       <origin xyz="0 0 0" rpy="0 0 0" />
       <geometry>
-        <!--<box size="0.55 0.32 0.155" />-->
+        <!--<box size="${base_link_length} ${base_link_width} ${base_link_height}" />-->
         <mesh filename="package://volksbot_driver/meshes/base.stl"/>
       </geometry>
     </collision>
-    <xacro:box_inertial x="0.55" y="0.32" z="0.155" mass="${base_mass}"/>
+    <xacro:box_inertial x="${base_link_length}" y="${base_link_width}" z="${base_link_height}" mass="${base_mass}"/>
   </link>
   <xacro:macro name="volksbot_wheel" params="name xyz rotate_visual">

Commit message: remove fake inertial from /base_footprint
KDL complained about it and gazebo still seems to work
as expected. Looks like the comment was out of date.

File: urdf/volksbot.urdf.xacro (robot description, xacro)
@@ -84,15 +84,6 @@
   <xacro:volksbot_wheel name="right_rear" xyz="${-wheel_x_offset} ${-axis_length/2} ${wheel_z_offset}" rotate_visual="0" />
   <!-- base_footprint is a fictitious link(frame) that is on the ground right below base_link origin,
-       navigation stack dedpends on this frame -->
-  <link name="base_footprint">
-    <!-- this needs to have a fake inertial element, otherwise all children will be ignored by Gazebo -->
-    <inertial>
-      <mass value="0.0001" />
-      <origin xyz="0 0 0" />
-      <inertia ixx="0.0001" ixy="0.0" ixz="0.0"
-        iyy="0.0001" iyz="0.0"
-        izz="0.0001" />
-    </inertial>
-  </link>
+       navigation stack depends on this frame -->
+  <link name="base_footprint"/>
   <joint name="base_footprint_joint" type="fixed">
     <!-- base link has 5cm clearence from ground and height of 15.5cm -->

Commit message: urdf: removed common.xacro
This was just a copy of uos_common_urdf/common.xacro. We copied that
here because we don't want to depend on another stack just for that
file; however, keeping the two consistent is too much of a hassle, so
I've just expanded the macros into the URDF.

Conflicts:
	urdf/volksbot.urdf.xacro

File: urdf/volksbot.urdf.xacro (robot description, xacro)
@@ -5,5 +5,5 @@
   xmlns:xacro="http://ros.org/wiki/xacro"
   name="volksbot_base">
-  <include filename="$(find volksbot_driver)/urdf/common.xacro" />
+  <xacro:property name="M_PI" value="3.1415926535897931" />
   <xacro:property name="wheel_width" value="0.06" />
   <xacro:property name="wheel_radius" value="0.0985" />
@@ -35,5 +35,11 @@
       </geometry>
     </collision>
-    <xacro:box_inertial x="${base_link_length}" y="${base_link_width}" z="${base_link_height}" mass="${base_mass}"/>
+    <inertial>
+      <mass value="${base_mass}" />
+      <origin xyz="0 0 0" />
+      <inertia ixx="${0.0833333 * base_mass * (base_link_width*base_link_width + base_link_height*base_link_height)}" ixy="0.0" ixz="0.0"
+        iyy="${0.0833333 * base_mass * (base_link_length*base_link_length + base_link_height*base_link_height)}" iyz="0.0"
+        izz="${0.0833333 * base_mass * (base_link_length*base_link_length + base_link_width*base_link_width)}" />
+    </inertial>
   </link>
   <xacro:macro name="volksbot_wheel" params="name xyz rotate_visual">
@@ -59,5 +65,11 @@
         </geometry>
       </collision>
-      <xacro:cylinder_inertial radius="${wheel_radius}" length="${wheel_width}" mass="${wheel_mass}"/>
+      <inertial>
+        <mass value="${wheel_mass}" />
+        <origin xyz="0 0 0" />
+        <inertia ixx="${0.0833333 * wheel_mass * (3 * wheel_radius * wheel_radius + wheel_width * wheel_width)}" ixy="0.0" ixz="0.0"
+          iyy="${0.0833333 * wheel_mass * (3 * wheel_radius * wheel_radius + wheel_width * wheel_width)}" iyz="0.0"
+          izz="${0.5 * wheel_mass * wheel_radius * wheel_radius}" />
+      </inertial>
     </link>
     <!-- friction parameters -->

Commit message: urdf: removed common.xacro
This was just a copy of uos_common_urdf/common.xacro. We copied that
here because we don't want to depend on another stack just for that
file; however, keeping the two consistent is too much of a hassle, so
I've just expanded the macros into the URDF.

File: urdf/volksbot.urdf.xacro (robot description, xacro)
@@ -5,5 +5,5 @@
   xmlns:xacro="http://ros.org/wiki/xacro"
   name="volksbot_base">
-  <xacro:include filename="$(find volksbot_driver)/urdf/common.xacro" />
+  <xacro:property name="M_PI" value="3.1415926535897931" />
   <xacro:property name="wheel_width" value="0.06" />
   <xacro:property name="wheel_radius" value="0.0985" />
@@ -35,5 +35,11 @@
       </geometry>
     </collision>
-    <xacro:box_inertial x="${base_link_length}" y="${base_link_width}" z="${base_link_height}" mass="${base_mass}"/>
+    <inertial>
+      <mass value="${base_mass}" />
+      <origin xyz="0 0 0" />
+      <inertia ixx="${0.0833333 * base_mass * (base_link_width*base_link_width + base_link_height*base_link_height)}" ixy="0.0" ixz="0.0"
+        iyy="${0.0833333 * base_mass * (base_link_length*base_link_length + base_link_height*base_link_height)}" iyz="0.0"
+        izz="${0.0833333 * base_mass * (base_link_length*base_link_length + base_link_width*base_link_width)}" />
+    </inertial>
   </link>
   <xacro:macro name="volksbot_wheel" params="name xyz rotate_visual">
@@ -59,5 +65,11 @@
         </geometry>
       </collision>
-      <xacro:cylinder_inertial radius="${wheel_radius}" length="${wheel_width}" mass="${wheel_mass}"/>
+      <inertial>
+        <mass value="${wheel_mass}" />
+        <origin xyz="0 0 0" />
+        <inertia ixx="${0.0833333 * wheel_mass * (3 * wheel_radius * wheel_radius + wheel_width * wheel_width)}" ixy="0.0" ixz="0.0"
+          iyy="${0.0833333 * wheel_mass * (3 * wheel_radius * wheel_radius + wheel_width * wheel_width)}" iyz="0.0"
+          izz="${0.5 * wheel_mass * wheel_radius * wheel_radius}" />
+      </inertial>
     </link>
     <!-- friction parameters -->

Commit message: urdf: changed the radius of the wheels

File: urdf/volksbot.urdf.xacro (robot description, xacro)
@@ -7,5 +7,5 @@
   <xacro:property name="M_PI" value="3.1415926535897931" />
   <xacro:property name="wheel_width" value="0.06" />
-  <xacro:property name="wheel_radius" value="0.0985" />
+  <xacro:property name="wheel_radius" value="0.103" />
   <xacro:property name="axis_length" value="0.41" />
   <xacro:property name="wheel_x_offset" value="0.225" />

Commit message: urdf: changed the way the z-coordinate of base_link is calculated
Note the commit 2d89c0.
Note that the base link is 3 mm heighter than it was before.

File: urdf/volksbot.urdf.xacro (robot description, xacro)
@@ -99,6 +99,5 @@
   <link name="base_footprint"/>
   <joint name="base_footprint_joint" type="fixed">
-    <!-- base link has 5cm clearence from ground and height of 15.5cm -->
-    <origin xyz="0 0 ${0.155/2 + 0.05}" rpy="0 0 0" />
+    <origin xyz="0 0 ${wheel_radius -  wheel_z_offset}" rpy="0 0 0" />
     <parent link="base_footprint"/>
     <child link="base_link" />

Commit message: urdf: changed the way the z-coordinate of base_link is calculated
Note the commit 2d89c0.
Note that the base link is 3 mm heighter than it was before.

File: urdf/volksbot.urdf.xacro (robot description, xacro)
@@ -108,6 +108,5 @@
   </link>
   <joint name="base_footprint_joint" type="fixed">
-    <!-- base link has 5cm clearence from ground and height of 15.5cm -->
-    <origin xyz="0 0 ${0.155/2 + 0.05}" rpy="0 0 0" />
+    <origin xyz="0 0 ${wheel_radius -  wheel_z_offset}" rpy="0 0 0" />
     <parent link="base_footprint"/>
     <child link="base_link" />

Commit message: urdf: added new link "base_top"
base_top is at the top of the base, above base_link.

File: urdf/volksbot.urdf.xacro (robot description, xacro)
@@ -103,4 +103,10 @@
     <child link="base_link" />
   </joint>
+  <link name="base_top" />
+  <joint name="base_top_joint" type="fixed">
+    <origin xyz="0 0 ${base_link_height / 2.0}" rpy="0 0 0" />
+    <parent link="base_link" />
+    <child link="base_top"/>
+  </joint>
   <gazebo>
     <plugin name="volksbot_diffdrive" filename="libgazebo_ros_diffdrive_uos.so">

Commit message: urdf: added new link "base_top"
base_top is at the top of the base, above base_link.

File: urdf/volksbot.urdf.xacro (robot description, xacro)
@@ -112,4 +112,10 @@
     <child link="base_link" />
   </joint>
+  <link name="base_top" />
+  <joint name="base_top_joint" type="fixed">
+    <origin xyz="0 0 ${base_link_height / 2.0}" rpy="0 0 0" />
+    <parent link="base_link" />
+    <child link="base_top"/>
+  </joint>
   <gazebo>
     <controller:gazebo_ros_diffdrive_uos name="volksbot_diffdrive" plugin="libgazebo_ros_diffdrive_uos.so">

Commit message: volksbot URDF: reduce friction of front + rear wheels
This improves the turning behaviour and makes it a bit more realistic.

File: urdf/volksbot.urdf.xacro (robot description, xacro)
@@ -44,5 +44,5 @@
     </inertial>
   </link>
-  <xacro:macro name="volksbot_wheel" params="name xyz rotate_visual">
+  <xacro:macro name="volksbot_wheel" params="name xyz rotate_visual friction">
     <!-- rotate_visual: 0 for right side, 1 for left side -->
     <link name="${name}_wheel_link">
@@ -77,6 +77,6 @@
     <gazebo reference="${name}_wheel_link">
       <!-- Turtlebot: -->
-      <mu1 value="10"/>
-      <mu2 value="10"/>
+      <mu1 value="${friction}"/>
+      <mu2 value="${friction}"/>
       <kp value="100000000.0"/>
       <kd value="10000.0"/>
@@ -90,10 +90,10 @@
     </joint>
   </xacro:macro>
-  <xacro:volksbot_wheel name="left_front" xyz="${wheel_x_offset} ${axis_length/2} ${wheel_z_offset}" rotate_visual="1" />
-  <xacro:volksbot_wheel name="left_middle" xyz="0 ${axis_length/2} ${wheel_z_offset}" rotate_visual="1" />
-  <xacro:volksbot_wheel name="left_rear" xyz="${-wheel_x_offset} ${axis_length/2} ${wheel_z_offset}" rotate_visual="1" />
-  <xacro:volksbot_wheel name="right_front" xyz="${wheel_x_offset} ${-axis_length/2} ${wheel_z_offset}" rotate_visual="0" />
-  <xacro:volksbot_wheel name="right_middle" xyz="0 ${-axis_length/2} ${wheel_z_offset}" rotate_visual="0" />
-  <xacro:volksbot_wheel name="right_rear" xyz="${-wheel_x_offset} ${-axis_length/2} ${wheel_z_offset}" rotate_visual="0" />
+  <xacro:volksbot_wheel name="left_front" xyz="${wheel_x_offset} ${axis_length/2} ${wheel_z_offset}" rotate_visual="1" friction="1.0" />
+  <xacro:volksbot_wheel name="left_middle" xyz="0 ${axis_length/2} ${wheel_z_offset}" rotate_visual="1" friction="100.0" />
+  <xacro:volksbot_wheel name="left_rear" xyz="${-wheel_x_offset} ${axis_length/2} ${wheel_z_offset}" rotate_visual="1" friction="1.0" />
+  <xacro:volksbot_wheel name="right_front" xyz="${wheel_x_offset} ${-axis_length/2} ${wheel_z_offset}" rotate_visual="0" friction="1.0" />
+  <xacro:volksbot_wheel name="right_middle" xyz="0 ${-axis_length/2} ${wheel_z_offset}" rotate_visual="0" friction="100.0" />
+  <xacro:volksbot_wheel name="right_rear" xyz="${-wheel_x_offset} ${-axis_length/2} ${wheel_z_offset}" rotate_visual="0" friction="1.0" />
   <!-- base_footprint is a fictitious link(frame) that is on the ground right below base_link origin,
        navigation stack depends on this frame -->

Commit message: volksbot URDF: reduce friction of front + rear wheels
This improves the turning behaviour and makes it a bit more realistic.

File: urdf/volksbot.urdf.xacro (robot description, xacro)
@@ -44,5 +44,5 @@
     </inertial>
   </link>
-  <xacro:macro name="volksbot_wheel" params="name xyz rotate_visual">
+  <xacro:macro name="volksbot_wheel" params="name xyz rotate_visual friction">
     <!-- rotate_visual: 0 for right side, 1 for left side -->
     <link name="${name}_wheel_link">
@@ -77,6 +77,6 @@
     <gazebo reference="${name}_wheel_link">
       <!-- Turtlebot: -->
-      <mu1 value="10"/>
-      <mu2 value="10"/>
+      <mu1 value="${friction}"/>
+      <mu2 value="${friction}"/>
       <kp value="100000000.0"/>
       <kd value="10000.0"/>
@@ -90,10 +90,10 @@
     </joint>
   </xacro:macro>
-  <xacro:volksbot_wheel name="left_front" xyz="${wheel_x_offset} ${axis_length/2} ${wheel_z_offset}" rotate_visual="1" />
-  <xacro:volksbot_wheel name="left_middle" xyz="0 ${axis_length/2} ${wheel_z_offset}" rotate_visual="1" />
-  <xacro:volksbot_wheel name="left_rear" xyz="${-wheel_x_offset} ${axis_length/2} ${wheel_z_offset}" rotate_visual="1" />
-  <xacro:volksbot_wheel name="right_front" xyz="${wheel_x_offset} ${-axis_length/2} ${wheel_z_offset}" rotate_visual="0" />
-  <xacro:volksbot_wheel name="right_middle" xyz="0 ${-axis_length/2} ${wheel_z_offset}" rotate_visual="0" />
-  <xacro:volksbot_wheel name="right_rear" xyz="${-wheel_x_offset} ${-axis_length/2} ${wheel_z_offset}" rotate_visual="0" />
+  <xacro:volksbot_wheel name="left_front" xyz="${wheel_x_offset} ${axis_length/2} ${wheel_z_offset}" rotate_visual="1" friction="1.0" />
+  <xacro:volksbot_wheel name="left_middle" xyz="0 ${axis_length/2} ${wheel_z_offset}" rotate_visual="1" friction="100.0" />
+  <xacro:volksbot_wheel name="left_rear" xyz="${-wheel_x_offset} ${axis_length/2} ${wheel_z_offset}" rotate_visual="1" friction="1.0" />
+  <xacro:volksbot_wheel name="right_front" xyz="${wheel_x_offset} ${-axis_length/2} ${wheel_z_offset}" rotate_visual="0" friction="1.0" />
+  <xacro:volksbot_wheel name="right_middle" xyz="0 ${-axis_length/2} ${wheel_z_offset}" rotate_visual="0" friction="100.0" />
+  <xacro:volksbot_wheel name="right_rear" xyz="${-wheel_x_offset} ${-axis_length/2} ${wheel_z_offset}" rotate_visual="0" friction="1.0" />
   <!-- base_footprint is a fictitious link(frame) that is on the ground right below base_link origin,
        navigation stack dedpends on this frame -->

Commit message: added thomas' ros2 driver to humble branch

File: urdf/volksbot.urdf.xacro (robot description, xacro)
@@ -13,5 +13,5 @@
   <xacro:property name="wheel_z_offset" value="-0.0275" />
   <xacro:property name="turning_adaptation" value="0.95" />
-  <xacro:property name="base_mass" value="10" />
+  <xacro:property name="base_mass" value="10.001" />
   <xacro:property name="wheel_mass" value="0.25" />
   <xacro:property name="base_link_length" value="0.55"/>
@@ -23,5 +23,5 @@
       <geometry>
         <!--<box size="${base_link_length} ${base_link_width} ${base_link_height}" />-->
-        <mesh filename="package://volksbot_driver/meshes/base.stl"/>
+        <mesh filename="file://$(find volksbot_driver)/meshes/base.stl"/>
       </geometry>
       <material name="grey" >
@@ -33,5 +33,5 @@
       <geometry>
         <!--<box size="${base_link_length} ${base_link_width} ${base_link_height}" />-->
-        <mesh filename="package://volksbot_driver/meshes/base.stl"/>
+        <mesh filename="file://$(find volksbot_driver)/meshes/base.stl"/>
       </geometry>
     </collision>
@@ -51,5 +51,5 @@
         <geometry>
           <!--<cylinder length="${wheel_width}" radius="${wheel_radius}"/>-->
-          <mesh filename="package://volksbot_driver/meshes/wheel.stl" />
+          <mesh filename="file://$(find volksbot_driver)/meshes/wheel.stl" />
         </geometry>
         <material name="blackish">
@@ -63,5 +63,5 @@
           <!-- using STL for collision to fix http://answers.ros.org/question/2368/gazebo-model-wheels-slip-after-upgrade-to-electric -->
           <!--<cylinder length="${wheel_width}" radius="${wheel_radius}"/>-->
-          <mesh filename="package://volksbot_driver/meshes/wheel.stl" />
+          <mesh filename="file://$(find volksbot_driver)/meshes/wheel.stl" />
         </geometry>
       </collision>
